File: pico_buck_board/pico_buck_board.kicad_sch (KiCad schematic)
At the start: 7 parts, among them J101 Conn_01x02, J102 part_of_pico, J103 Conn_01x02, J104 Conn_01x02, J105 Conn_01x02, Q101 Q_PMOS_SSSGDDDD

Commit message: add footprints
Parts:
- removed Q101: Q_PMOS_SSSGDDDD, symbol good_things:Q_PMOS_SSSGDDDD
- removed R101: 10k, symbol Device:R
- added D101: PJON GGE, Diode_SMD:D_3220_8050Metric_Pad2.65x5.15mm_HandSolder, symbol Device:D
Connections:
- net GND: now also D101.2 (A)
- net vin renamed +5V
- net +5V: now also D101.1 (K)

Commit message: rev1 board done
Connections:
- net buck0_fb: now also J102.14 (Pin_14); no longer J102.11 (Pin_11)
- net buck0_sw0: now also J102.6 (Pin_6); no longer J102.1 (Pin_1)
- net buck0_sw1: now also J102.7 (Pin_7); no longer J102.2 (Pin_2)
- net buck1_fb: now also J102.11 (Pin_11); no longer J102.12 (Pin_12)
- net buck1_sw0: now also J102.1 (Pin_1); no longer J102.4 (Pin_4)
- net buck1_sw1: now also J102.2 (Pin_2); no longer J102.5 (Pin_5)
- net buck2_fb: now also J102.12 (Pin_12); no longer J102.14 (Pin_14)
- net buck2_sw0: now also J102.4 (Pin_4); no longer J102.6 (Pin_6)
- net buck2_sw1: now also J102.5 (Pin_5); no longer J102.7 (Pin_7)
Changed lines of the file:
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@@
     (effects (font (size 1.5875 1.5875)) (justify right bottom))
   )
-  (label "buck0_fb" (at 89.535 56.515 0)
+  (label "buck0_fb" (at 89.535 48.895 0)
     (effects (font (size 1.27 1.27)) (justify left bottom))
   )
@@
     (effects (font (size 1.27 1.27)) (justify left bottom))
   )
-  (label "buck2_sw1" (at 86.995 66.675 0)
+  (label "buck2_sw1" (at 86.995 71.755 0)
     (effects (font (size 1.27 1.27)) (justify left bottom))
   )
-  (label "buck2_sw0" (at 86.995 69.215 0)
+  (label "buck2_sw0" (at 86.995 74.295 0)
     (effects (font (size 1.27 1.27)) (justify left bottom))
   )
@@
     (effects (font (size 1.27 1.27)) (justify left bottom))
   )
-  (label "buck1_fb" (at 89.535 53.975 0)
+  (label "buck1_fb" (at 89.535 56.515 0)
     (effects (font (size 1.27 1.27)) (justify left bottom))
   )
@@
     (effects (font (size 1.27 1.27)) (justify left bottom))
   )
-  (label "buck0_sw0" (at 86.995 81.915 0)
+  (label "buck0_sw0" (at 86.995 69.215 0)
     (effects (font (size 1.27 1.27)) (justify left bottom))
   )
@@
     (effects (font (size 1.27 1.27)) (justify right bottom))
   )
-  (label "buck0_sw1" (at 86.995 79.375 0)
+  (label "buck0_sw1" (at 86.995 66.675 0)
     (effects (font (size 1.27 1.27)) (justify left bottom))
   )
-  (label "buck1_sw1" (at 86.995 71.755 0)
+  (label "buck1_sw1" (at 86.995 79.375 0)
     (effects (font (size 1.27 1.27)) (justify left bottom))
   )
@@
     (effects (font (size 1.27 1.27)) (justify left bottom))
   )
-  (label "buck1_sw0" (at 86.995 74.295 0)
+  (label "buck1_sw0" (at 86.995 81.915 0)
     (effects (font (size 1.27 1.27)) (justify left bottom))
   )
-  (label "buck2_fb" (at 89.535 48.895 0)
+  (label "buck2_fb" (at 89.535 53.975 0)
     (effects (font (size 1.27 1.27)) (justify left bottom))
   )
