File: pico_buck_board/sync_buck.kicad_sch (KiCad schematic)
At the start: 18 parts, among them Q201 Q_PMOS_SSSGDDDD, Q202 Q_PMOS_SSSGDDDD

Commit message: add footprints
Parts:
- removed D201: D_Schottky, symbol Device:D_Schottky
- removed Q201: Q_PMOS_SSSGDDDD, symbol good_things:Q_PMOS_SSSGDDDD
- added D201: PJON GGE, Diode_SMD:D_3220_8050Metric_Pad2.65x5.15mm_HandSolder, symbol Device:D
- added Q201, Q203: KST5551MTF, Package_TO_SOT_SMD:SOT-23, symbol Device:Q_NPN_BEC
- added Q204: FSD4435, Package_SO:SO-8_3.9x4.9mm_P1.27mm, symbol good_things:Q_PMOS_SSSGDDDD
- added R203, R204: 10, symbol Device:R
- L202: footprint Inductor_SMD:L_Wuerth_HCI-1350 -> Inductor_SMD:L_Bourns_SRR1210A
- Q202: value Q_PMOS_SSSGDDDD -> FSD4435; footprint (none) -> Package_SO:SO-8_3.9x4.9mm_P1.27mm
- R201, R202: value 100 -> 1k
Connections:
- net GND: now also D201.2 (A), Q201.2 (E), Q203.2 (E), Q204.1 (S), Q204.2 (S), Q204.3 (S); no longer Q202.1 (S), Q202.2 (S), Q202.3 (S)
- net Vin: now also Q202.1 (S), Q202.2 (S), Q202.3 (S), R203.2, R204.2
- net sw0: now also R201.2; no longer R201.1
- net sw1: now also R202.2; no longer R202.1
- net swr0: now also R201.1, Q201.1 (B); no longer R201.2
- net swr1: now also R202.1, Q203.1 (B); no longer Q202.4 (G), R202.2
- net vsw: now also Q202.5 (D), Q202.6 (D), Q202.7 (D), Q202.8 (D)
- net vsw_d: now also D201.1 (K)
- net vsw_fet: now also Q204.5 (D), Q204.6 (D), Q204.7 (D), Q204.8 (D); no longer Q202.5 (D), Q202.6 (D), Q202.7 (D), Q202.8 (D)
- new net sw1_gate: Q201.3 (C), Q202.4 (G), Q203.3 (C), Q204.4 (G), R203.1, R204.1

Commit message: some layoutin'
Parts:
- JP301: renamed from JP201; footprint (none) -> Jumper:SolderJumper-3_P1.3mm_Open_Pad1.0x1.5mm
- JP302: renamed from JP202; footprint (none) -> Jumper:SolderJumper-3_P1.3mm_Open_Pad1.0x1.5mm
- R301: renamed from R201; footprint (none) -> Resistor_SMD:R_0603_1608Metric_Pad0.98x0.95mm_HandSolder
- R302: renamed from R202; footprint (none) -> Resistor_SMD:R_0603_1608Metric_Pad0.98x0.95mm_HandSolder
- R303: renamed from R203; footprint (none) -> Resistor_SMD:R_0603_1608Metric_Pad0.98x0.95mm_HandSolder
- R304: renamed from R204; footprint (none) -> Resistor_SMD:R_0603_1608Metric_Pad0.98x0.95mm_HandSolder
- renumbered C201 to C301, C202 to C302, C203 to C303, C204 to C304, C205 to C305, C206 to C306, C207 to C307, C208 to C308, D201 to D301, L201 to L301, L202 to L302, L203 to L303, Q201 to Q301, Q202 to Q302, Q203 to Q303, Q204 to Q304
Connections:
- net sw1_gate: no longer Q301.3 (C), Q302.4 (G), R303.1
- new net sw0_gate: Q301.3 (C), Q302.4 (G), R303.1

Commit message: rev1 board done
Parts:
- renumbered C301 to C401, C302 to C402, C303 to C403, C304 to C404, C305 to C405, C306 to C406, C307 to C407, C308 to C408, D301 to D401, JP301 to JP401, JP302 to JP402, L301 to L401, L302 to L402, L303 to L403, Q301 to Q401, Q302 to Q402, Q303 to Q403, Q304 to Q404, R301 to R401, R302 to R402, R303 to R403, R304 to R404
