File: pico_buck_board/pico_buck_board.kicad_pcb (KiCad board)
At the start: 2 copper layers, 72 parts, among them J101 Conn_01x02, J102 part_of_pico, J103 Conn_01x02, J104 Conn_01x02, J105 Conn_01x02, Q201 KST5551MTF, Q202 FSD4435, Q203 KST5551MTF, Q204 FSD4435, Q301 KST5551MTF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

Commit message: rev1 board done
Parts:
- J102: moved to F.Cu
- moved R203 153.3 mm to (107.0, 31.0), turned to 90 degrees
- moved C202 151.4 mm to (105.3, 31.0), turned to -90 degrees
- moved C203 149.1 mm to (103.6, 31.0), turned to -90 degrees
- moved Q202 142.0 mm to (112.0, 30.0)
- moved R202 134.4 mm to (114.4, 17.0), turned to 90 degrees
- moved C201 133.3 mm to (96.0, 34.0), turned to -90 degrees
- moved Q203 132.3 mm to (118.0, 17.0), turned to 90 degrees
- moved R204 128.5 mm to (114.3, 20.4), turned to 180 degrees
- moved R201 128.4 mm to (109.0, 35.0), turned to 90 degrees
- moved Q204 122.6 mm to (120.0, 23.0), turned to -90 degrees
- moved Q201 121.1 mm to (112.0, 35.0), turned to 90 degrees
- moved C205 119.4 mm to (141.0, 32.9), turned to -90 degrees
- moved JP202 116.0 mm to (125.0, 30.0), turned to 90 degrees
- moved JP201 109.8 mm to (120.0, 30.0), turned to 90 degrees
- moved L202 108.7 mm to (135.0, 24.0)
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Connections:
- J102 pad 1: /buck0_sw0 -> /buck1_sw0
- J102 pad 11: /buck0_fb -> /buck1_fb
- J102 pad 12: /buck1_fb -> /buck2_fb
- J102 pad 14: /buck2_fb -> /buck0_fb
- J102 pad 2: /buck0_sw1 -> /buck1_sw1
- J102 pad 4: /buck1_sw0 -> /buck2_sw0
- J102 pad 5: /buck1_sw1 -> /buck2_sw1
- J102 pad 6: /buck2_sw0 -> /buck0_sw0
- J102 pad 7: /buck2_sw1 -> /buck0_sw1
Routing:
- net /buck0_sw1: track 0.00 -> 139.7 mm, vias 0 -> 1
- net /buck0_sw0: track 0.00 -> 130.7 mm, vias 0 -> 1
- net /buck2_sw1: track 0.00 -> 117.5 mm, vias 0 -> 1
- net /buck2_sw0: track 2.38 -> 106.2 mm
- net /buck1_sw0: track 1.59 -> 94.3 mm
- net /buck1_sw1: track 0.00 -> 92.3 mm, vias 0 -> 1
- net /buck1_fb: track 3.48 -> 69.1 mm
- net /buck2_fb: track 3.88 -> 46.9 mm
- net /buck0_fb: track 0.00 -> 18.5 mm, vias 0 -> 1
- net GND: track 0.00 -> 10.1 mm, vias 0 -> 3
- net /sync_buck/sw1_gate: track 0.00 -> 7.29 mm
- net /sync_buck/sw0_gate: track 0.00 -> 5.90 mm
- net /sync_buck/swr1: track 0.00 -> 2.66 mm
- net /sync_buck/swr0: track 0.00 -> 2.06 mm
- added copper zone on F.Cu, net /buck0_out
- added copper zone on F.Cu, net /sync_buck/vsw
- added copper zone on F.Cu, net /sync_buck/vsw_d
- added copper zone on F.Cu, net /sync_buck/vsw_fet
- added copper zone on F.Cu, net /sync_buck/vsw_lbig
- added copper zone on F.Cu, net /sync_buck/vsw_lsmall
- added copper zone on B.Cu, net GND
Other:
- board outline added: 89.4 x 88.2 mm
- board text added: "ANTON LÖÖF REV1 2022"
- board text added: "B0 GND"
- board text added: "B1 GND"
- board text added: "B2 GND"
- board text added: "SolderJumper_3_Open"
- board text added: "VIN GND"
- board text added: "b0_fb gnd b2_fb b1_fb nc nc gnd b0_sw1 b0_sw0 b2_sw1 b2_sw0 gnd b1_sw1 b1_sw0"
- board text added: "pico_buck"

Commit message: add spwm sw
Parts:
- moved C203 131.5 mm to (204.3, 115.5)
- moved C208 131.5 mm to (251.4, 104.4)
- moved J102 131.5 mm to (267.1, 136.8)
- moved C201 131.5 mm to (196.7, 118.5)
- moved C202 131.5 mm to (206.0, 115.5)
- moved C204 131.5 mm to (244.0, 117.4)
- moved C205 131.5 mm to (241.7, 117.4)
- moved C206 131.5 mm to (251.7, 119.5)
- moved C207 131.5 mm to (245.7, 104.5)
- moved C301 131.5 mm to (196.5, 177.2)
- moved C302 131.5 mm to (203.5, 174.2)
- moved C303 131.5 mm to (205.5, 174.2)
- moved C304 131.5 mm to (243.5, 176.3)
- moved C305 131.5 mm to (241.5, 176.2)
- moved C306 131.5 mm to (251.5, 178.2)
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